Commit message: update new model

File: gm_description/urdf/gold_miner_robot.urdf (robot description, URDF)
Before this commit: robot gold_miner_robot, 6 links, 5 joints
Links:
- link base: geometry collision mesh filename=package://gm_description/meshes/base.STL; visual mesh filename=package://gm_description/meshes/base.STL
- link base_joint: geometry collision mesh filename=package://gm_description/meshes/base_joint.STL; visual mesh filename=package://gm_description/meshes/base_joint.STL
- link elbow_joint: geometry collision mesh filename=package://gm_description/meshes/elbow_joint.STL; visual mesh filename=package://gm_description/meshes/elbow_joint.STL
- link shoulder_joint: geometry collision mesh filename=package://gm_description/meshes/shoulder_joint.STL; visual mesh filename=package://gm_description/meshes/shoulder_joint.STL
- link wrist_joint_1: geometry collision mesh filename=package://gm_description/meshes/wrist_joint_1.STL; visual mesh filename=package://gm_description/meshes/wrist_joint_1.STL
- link wrist_joint_2: geometry collision mesh filename=package://gm_description/meshes/wrist_joint_2.STL; visual mesh filename=package://gm_description/meshes/wrist_joint_2.STL
Joints:
- joint elbow_joint: limit lower=3.14 upper=-3.14 effort=150 velocity=5 -> lower=-3.14 upper=3.14 effort=150 velocity=5
